File: MoonBoard.kicad_pcb (KiCad board)
At the start: 2 copper layers, 3.6 x 3.3 mm, 541 parts, among them U1 AP2112K-3.3, U10 SLSS49E-3, U11 SLSS49E-3, U12 SLSS49E-3, U13 SLSS49E-3, U14 SLSS49E-3, U15 SLSS49E-3, U16 SLSS49E-3, U17 SLSS49E-3, U18 SLSS49E-3, U19 SLSS49E-3, U2 CD74HC4067M, U20 SLSS49E-3, U21 SLSS49E-3, U22 SLSS49E-3, U23 SLSS49E-3, U24 SLSS49E-3, U25 SLSS49E-3, U26 SLSS49E-3, U27 SLSS49E-3, U28 SLSS49E-3, U29 SLSS49E-3, U3 CD74HC4067M, U30 SLSS49E-3, U31 SLSS49E-3, U32 SLSS49E-3, U33 SLSS49E-3, U34 SLSS49E-3, U35 SLSS49E-3, U36 SLSS49E-3, U37 SLSS49E-3, U38 SLSS49E-3, U39 SLSS49E-3, U4 CD74HC4067M, U40 SLSS49E-3, U41 SLSS49E-3, U42 SLSS49E-3, U43 SLSS49E-3, U44 SLSS49E-3, U45 SLSS49E-3, U46 SLSS49E-3, U47 SLSS49E-3, U48 SLSS49E-3, U49 SLSS49E-3, U5 CD74HC4067M, U50 SLSS49E-3, U51 SLSS49E-3, U52 SLSS49E-3, U53 SLSS49E-3, U54 SLSS49E-3, U55 SLSS49E-3, U56 SLSS49E-3, U57 SLSS49E-3, U58 SLSS49E-3, U59 SLSS49E-3, U6 STM32F446RETx, U60 SLSS49E-3, U61 SLSS49E-3, U62 SLSS49E-3, U63 SLSS49E-3, U64 SLSS49E-3, U65 SLSS49E-3, U66 SLSS49E-3, U67 SLSS49E-3, U68 SLSS49E-3, U69 SLSS49E-3, U7 CD74HC4067M, U70 SLSS49E-3, U71 SLSS49E-3, U72 SLSS49E-3, U73 SLSS49E-3, U74 SLSS49E-3, U75 SLSS49E-3, U76 SLSS49E-3, U77 SLSS49E-3, U78 SLSS49E-3, U79 SLSS49E-3, U8 CD74HC4067M, U80 SLSS49E-3, U81 SLSS49E-3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

Commit message: switch layout
Parts:
- removed S1, S3: MX_stab, PCM_marbastlib-mx:STAB_MX_ISO
- removed S2: STAB_MX_ISO, PCM_marbastlib-mx:STAB_MX_ISO
- removed S4: MX_stab, PCM_marbastlib-mx:STAB_MX_P_6.25u
- removed U10, U11, U12, U13, U14, U15, U16, U17, U18, U19, U20, U21, U22, U23, U24, U25, U26, U27, U28, U29, U30, U31, U32, U33, U34, U35, U36, U37, U38, U39, U40, U41, U42, U43, U44, U45, U46, U47, U48, U49, U50, U51, U52, U53, U54, U55, U56, U57, U58, U59, U60, U61, U62, U63, U64, U65, U66, U67, U68, U69, U70, U71, U72, U73, U74, U75, U76, U77, U78, U79, U80, U81, U82, U83, U84, U85, U86, U87, U88, U89, U9: SLSS49E-3, MoonBoard:SLSS49E-3 with MX holes
- added C271: 100n, Capacitor_SMD:C_0402_1005Metric, F.Cu at (251.4, -113.4)
- added C272: 100n, Capacitor_SMD:C_0402_1005Metric, F.Cu at (251.4, -111.4)
- added C273: 100n, Capacitor_SMD:C_0402_1005Metric, F.Cu at (251.4, -109.4)
- added HALL1: SLSS49E-3, MoonBoard:SLSS49E-3 with MX holes, B.Cu at (42.9, 81.0)
- added HALL10: SLSS49E-3, MoonBoard:SLSS49E-3 with MX holes, B.Cu at (233.4, 81.0)
- added HALL11: SLSS49E-3, MoonBoard:SLSS49E-3 with MX holes, B.Cu at (252.4, 81.0)
- added HALL12: SLSS49E-3, MoonBoard:SLSS49E-3 with MX holes, B.Cu at (271.5, 81.0)
- added HALL13: SLSS49E-3, MoonBoard:SLSS49E-3 with MX holes, B.Cu at (290.5, 81.0)
- added HALL14: SLSS49E-3, MoonBoard:SLSS49E-3 with MX holes, B.Cu at (42.9, 104.8)
- added HALL15: SLSS49E-3, MoonBoard:SLSS49E-3 with MX holes, B.Cu at (61.9, 104.8)
- added HALL16: SLSS49E-3, MoonBoard:SLSS49E-3 with MX holes, B.Cu at (81.0, 104.8)
- added HALL17: SLSS49E-3, MoonBoard:SLSS49E-3 with MX holes, B.Cu at (100.0, 104.8)
- added HALL18: SLSS49E-3, MoonBoard:SLSS49E-3 with MX holes, B.Cu at (119.1, 104.8)
- added HALL19: SLSS49E-3, MoonBoard:SLSS49E-3 with MX holes, B.Cu at (138.1, 104.8)
- added HALL2: SLSS49E-3, MoonBoard:SLSS49E-3 with MX holes, B.Cu at (71.4, 81.0)
- added HALL20: SLSS49E-3, MoonBoard:SLSS49E-3 with MX holes, B.Cu at (157.2, 104.8)
- added HALL21: SLSS49E-3, MoonBoard:SLSS49E-3 with MX holes, B.Cu at (176.2, 104.8)
- added HALL22: SLSS49E-3, MoonBoard:SLSS49E-3 with MX holes, B.Cu at (195.3, 104.8)
- added HALL23: SLSS49E-3, MoonBoard:SLSS49E-3 with MX holes, B.Cu at (214.3, 104.8)
- added HALL24: SLSS49E-3, MoonBoard:SLSS49E-3 with MX holes, B.Cu at (233.4, 104.8)
- added HALL25: SLSS49E-3, MoonBoard:SLSS49E-3 with MX holes, B.Cu at (252.4, 104.8)
- added HALL26: SLSS49E-3, MoonBoard:SLSS49E-3 with MX holes, B.Cu at (271.5, 104.8)
- added HALL27: SLSS49E-3, MoonBoard:SLSS49E-3 with MX holes, B.Cu at (300.0, 104.8)
- added HALL28: SLSS49E-3, MoonBoard:SLSS49E-3 with 1.5u MX holes, B.Cu at (47.6, 123.8)
- added HALL29: SLSS49E-3, MoonBoard:SLSS49E-3 with MX holes, B.Cu at (71.4, 123.8)
- added HALL3: SLSS49E-3, MoonBoard:SLSS49E-3 with MX holes, B.Cu at (90.5, 81.0)
- added HALL30: SLSS49E-3, MoonBoard:SLSS49E-3 with MX holes, B.Cu at (90.5, 123.8)
- added HALL31: SLSS49E-3, MoonBoard:SLSS49E-3 with MX holes, B.Cu at (109.5, 123.8)
- added HALL32: SLSS49E-3, MoonBoard:SLSS49E-3 with MX holes, B.Cu at (128.6, 123.8)
- added HALL33: SLSS49E-3, MoonBoard:SLSS49E-3 with MX holes, B.Cu at (147.6, 123.8)
- added HALL34: SLSS49E-3, MoonBoard:SLSS49E-3 with MX holes, B.Cu at (166.7, 123.8)
- added HALL35: SLSS49E-3, MoonBoard:SLSS49E-3 with MX holes, B.Cu at (185.7, 123.8)
- added HALL36: SLSS49E-3, MoonBoard:SLSS49E-3 with MX holes, B.Cu at (204.8, 123.8)
- added HALL37: SLSS49E-3, MoonBoard:SLSS49E-3 with MX holes, B.Cu at (223.8, 123.8)
- added HALL38: SLSS49E-3, MoonBoard:SLSS49E-3 with MX holes, B.Cu at (242.9, 123.8)
- added HALL39: SLSS49E-3, MoonBoard:SLSS49E-3 with MX holes, B.Cu at (261.9, 123.8)
- added HALL4: SLSS49E-3, MoonBoard:SLSS49E-3 with MX holes, B.Cu at (109.5, 81.0)
- added HALL40: SLSS49E-3, MoonBoard:SLSS49E-3 with MX holes, B.Cu at (281.0, 123.8)
- added HALL41: SLSS49E-3, MoonBoard:SLSS49E-3 with MX holes, B.Cu at (307.2, 133.3)
- added HALL42: SLSS49E-3, MoonBoard:SLSS49E-3 with MX holes, B.Cu at (338.1, 123.8)
- added HALL43: SLSS49E-3, MoonBoard:SLSS49E-3 with 1.75u MX holes, B.Cu at (50.0, 142.9)
- added HALL44: SLSS49E-3, MoonBoard:SLSS49E-3 with MX holes, B.Cu at (76.2, 142.9)
- added HALL45: SLSS49E-3, MoonBoard:SLSS49E-3 with MX holes, B.Cu at (95.2, 142.9)
- added HALL46: SLSS49E-3, MoonBoard:SLSS49E-3 with MX holes, B.Cu at (114.3, 142.9)
- added HALL47: SLSS49E-3, MoonBoard:SLSS49E-3 with MX holes, B.Cu at (133.3, 142.9)
- added HALL48: SLSS49E-3, MoonBoard:SLSS49E-3 with MX holes, B.Cu at (152.4, 142.9)
- added HALL49: SLSS49E-3, MoonBoard:SLSS49E-3 with MX holes, B.Cu at (171.4, 142.9)
- added HALL5: SLSS49E-3, MoonBoard:SLSS49E-3 with MX holes, B.Cu at (128.6, 81.0)
- added HALL50: SLSS49E-3, MoonBoard:SLSS49E-3 with MX holes, B.Cu at (190.5, 142.9)
- added HALL51: SLSS49E-3, MoonBoard:SLSS49E-3 with MX holes, B.Cu at (209.6, 142.9)
- added HALL52: SLSS49E-3, MoonBoard:SLSS49E-3 with MX holes, B.Cu at (228.6, 142.9)
- added HALL53: SLSS49E-3, MoonBoard:SLSS49E-3 with MX holes, B.Cu at (247.7, 142.9)
- added HALL54: SLSS49E-3, MoonBoard:SLSS49E-3 with MX holes, B.Cu at (266.7, 142.9)
- added HALL55: SLSS49E-3, MoonBoard:SLSS49E-3 with MX holes, B.Cu at (285.8, 142.9)
- added HALL56: SLSS49E-3, MoonBoard:SLSS49E-3 with MX holes, B.Cu at (338.1, 142.9)
- added HALL57: SLSS49E-3, MoonBoard:SLSS49E-3 with 1.25u MX holes, B.Cu at (45.2, 161.9)
- added HALL58: SLSS49E-3, MoonBoard:SLSS49E-3 with MX holes, B.Cu at (66.7, 161.9)
- added HALL59: SLSS49E-3, MoonBoard:SLSS49E-3 with MX holes, B.Cu at (85.7, 161.9)
- added HALL6: SLSS49E-3, MoonBoard:SLSS49E-3 with MX holes, B.Cu at (152.4, 81.0)
- added HALL60: SLSS49E-3, MoonBoard:SLSS49E-3 with MX holes, B.Cu at (104.8, 161.9)
- added HALL61: SLSS49E-3, MoonBoard:SLSS49E-3 with MX holes, B.Cu at (123.8, 161.9)
- added HALL62: SLSS49E-3, MoonBoard:SLSS49E-3 with MX holes, B.Cu at (142.9, 161.9)
- added HALL63: SLSS49E-3, MoonBoard:SLSS49E-3 with MX holes, B.Cu at (161.9, 161.9)
- added HALL64: SLSS49E-3, MoonBoard:SLSS49E-3 with MX holes, B.Cu at (181.0, 161.9)
- added HALL65: SLSS49E-3, MoonBoard:SLSS49E-3 with MX holes, B.Cu at (200.0, 161.9)
- added HALL66: SLSS49E-3, MoonBoard:SLSS49E-3 with MX holes, B.Cu at (219.1, 161.9)
- added HALL67: SLSS49E-3, MoonBoard:SLSS49E-3 with MX holes, B.Cu at (238.1, 161.9)
- added HALL68: SLSS49E-3, MoonBoard:SLSS49E-3 with MX holes, B.Cu at (257.2, 161.9)
- added HALL69: SLSS49E-3, MoonBoard:SLSS49E-3 with 1.75u MX holes, B.Cu at (283.4, 161.9)
- added HALL7: SLSS49E-3, MoonBoard:SLSS49E-3 with MX holes, B.Cu at (171.4, 81.0)
- added HALL70: SLSS49E-3, MoonBoard:SLSS49E-3 with MX holes, B.Cu at (338.1, 161.9)
- added HALL71: SLSS49E-3, MoonBoard:SLSS49E-3 with MX holes, B.Cu at (314.3, 166.7)
- added HALL72: SLSS49E-3, MoonBoard:SLSS49E-3 with 1.25u MX holes, B.Cu at (45.2, 181.0)
- added HALL73: SLSS49E-3, MoonBoard:SLSS49E-3 with 1.25u MX holes, B.Cu at (69.1, 181.0)
- added HALL74: SLSS49E-3, MoonBoard:SLSS49E-3 with 1.25u MX holes, B.Cu at (92.9, 181.0)
- added HALL75: SLSS49E-3, MoonBoard:SLSS49E-3 with MX holes, B.Cu at (164.3, 181.0)
- added HALL76: SLSS49E-3, MoonBoard:SLSS49E-3 with MX holes, B.Cu at (233.4, 181.0)
- added HALL77: SLSS49E-3, MoonBoard:SLSS49E-3 with MX holes, B.Cu at (252.4, 181.0)
- added HALL78: SLSS49E-3, MoonBoard:SLSS49E-3 with MX holes, B.Cu at (271.5, 181.0)
- added HALL79: SLSS49E-3, MoonBoard:SLSS49E-3 with MX holes, B.Cu at (295.3, 185.7)
- added HALL8: SLSS49E-3, MoonBoard:SLSS49E-3 with MX holes, B.Cu at (190.5, 81.0)
- added HALL80: SLSS49E-3, MoonBoard:SLSS49E-3 with MX holes, B.Cu at (314.3, 185.7)
- added HALL81: SLSS49E-3, MoonBoard:SLSS49E-3 with MX holes, B.Cu at (333.4, 185.7)
- added HALL82: SLSS49E-3, MoonBoard:SLSS49E-3 with 1.5u MX holes, B.Cu at (322.2, 16.9)
- added HALL83: SLSS49E-3, MoonBoard:SLSS49E-3 with 2.25 MX holes, B.Cu at (297.6, 142.8)
- added HALL84: SLSS49E-3, MoonBoard:SLSS49E-3 with 2.25 MX holes, B.Cu at (54.7, 161.9)
- added HALL9: SLSS49E-3, MoonBoard:SLSS49E-3 with MX holes, B.Cu at (209.6, 81.0)
- added R88: 10k, Resistor_SMD:R_0402_1005Metric, F.Cu at (248.5, -113.4)
- added R89: 10k, Resistor_SMD:R_0402_1005Metric, F.Cu at (248.5, -111.4)
- added R90: 10k, Resistor_SMD:R_0402_1005Metric, F.Cu at (248.5, -109.4)
- added S27: STAB_MX_2u, PCM_marbastlib-mx:STAB_MX_2u, F.Cu at (300.0, 104.8)
- added S41: STAB_MX_ISO, PCM_marbastlib-mx:STAB_MX_ISO, F.Cu at (307.2, 133.3)
- added S75: STAB_MX_P_6.25U, PCM_marbastlib-mx:STAB_MX_P_6.25u, F.Cu at (164.3, 181.0)
- added S83: MX_stab, PCM_marbastlib-mx:STAB_MX_2.25u, F.Cu at (462.8, 107.2)
- added S84: MX_stab, PCM_marbastlib-mx:STAB_MX_2.25u, F.Cu at (54.8, 161.9)
- BOOT1, C1, C10, C100, C101, C102, C103, C104, C105, C106, C107, C108, C109, C11, C110, C111, C112, C113, C114, C115, C116, C117, C118, C119, C12, C120, C121, C122, C123, C124, C125, C126, C127, C128, C129, C13, C130, C131, C132, C133, C134, C135, C136, C137, C138, C139, C14, C140, C141, C142, C143, C144, C145, C146, C147, C148, C149, C15, C150, C151, C152, C153, C154, C155, C156, C157, C158, C159, C16, C160, C161, C162, C163, C164, C165, C166, C167, C168, C169, C17, C170, C171, C172, C173, C174, C175, C176, C177, C178, C179, C18, C180, C181, C182, C183, C184, C185, C186, C187, C188, C189, C19, C190, C191, C192, C193, C194, C195, C196, C197, C198, C199, C2, C20, C200, C201, C202, C203, C204, C205, C206, C207, C208, C209, C21, C210, C211, C212, C213, C214, C215, C216, C217, C218, C219, C22, C220, C221, C222, C223, C224, C225, C226, C227, C228, C229, C23, C230, C231, C232, C233, C234, C235, C236, C237, C238, C239, C24, C240, C241, C242, C243, C244, C245, C246, C247, C248, C249, C25, C250, C251, C252, C253, C254, C255, C256, C257, C258, C259, C26, C260, C261, C262, C263, C264, C265, C266, C267, C268, C269, C27, C270, C28, C29, C3, C30, C31, C32, C33, C34, C35, C36, C37, C38, C39, C4, C40, C41, C42, C43, C44, C45, C46, C47, C48, C49, C5, C50, C51, C52, C53, C54, C55, C56, C57, C58, C59, C6, C60, C61, C62, C63, C64, C65, C66, C67, C68, C69, C7, C70, C71, C72, C73, C74, C75, C76, C77, C78, C79, C8, C80, C81, C82, C83, C84, C85, C86, C87, C88, C89, C9, C90, C91, C92, C93, C94, C95, C96, C97, C98, C99, D1, ENCODER1, F1, LED1, LED10, LED11, LED12, LED13, LED14, LED15, LED16, LED17, LED18, LED19, LED2, LED20, LED21, LED22, LED23, LED24, LED25, LED26, LED27, LED28, LED29, LED3, LED30, LED31, LED32, LED33, LED34, LED35, LED36, LED37, LED38, LED39, LED4, LED40, LED41, LED42, LED43, LED44, LED45, LED46, LED47, LED48, LED49, LED5, LED50, LED51, LED52, LED53, LED54, LED55, LED56, LED57, LED58, LED59, LED6, LED60, LED61, LED62, LED63, LED64, LED65, LED66, LED67, LED68, LED69, LED7, LED70, LED71, LED72, LED73, LED74, LED75, LED76, LED77, LED78, LED79, LED8, LED80, LED81, LED9, OLED1, R1, R10, R11, R12, R13, R14, R15, R16, R17, R18, R19, R2, R20, R21, R22, R23, R24, R25, R26, R27, R28, R29, R3, R30, R31, R32, R33, R34, R35, R36, R37, R38, R39, R4, R40, R41, R42, R43, R44, R45, R46, R47, R48, R49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: moved to B.Cu
- moved C262 628.8 mm to (-50.9, -340.7), turned to 180 degrees
- moved C263 628.8 mm to (-50.9, -338.8), turned to 180 degrees
- moved C264 628.8 mm to (-50.9, -336.8), turned to 180 degrees
- moved C265 628.8 mm to (-50.9, -334.8), turned to 180 degrees
- moved C266 628.8 mm to (-50.9, -332.9), turned to 180 degrees
- moved C267 628.8 mm to (-50.9, -330.9), turned to 180 degrees
- moved C268 628.8 mm to (-50.9, -328.9), turned to 180 degrees
- moved C269 628.8 mm to (-50.9, -327.0), turned to 180 degrees
- moved C270 628.8 mm to (-50.9, -325.0), turned to 180 degrees
- moved C250 623.6 mm to (-48.1, -340.7), turned to 180 degrees
- moved C251 623.6 mm to (-48.1, -338.8), turned to 180 degrees
- moved C252 623.6 mm to (-48.1, -336.8), turned to 180 degrees
- moved C253 623.6 mm to (-48.1, -334.8), turned to 180 degrees
- moved C254 623.6 mm to (-48.1, -332.9), turned to 180 degrees
- moved C255 623.6 mm to (-48.1, -330.9), turned to 180 degrees
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Connections:
- U4 pad 16: unconnected-(U4-I15-Pad16) -> /F_KEYS_2_15
- U5 pad 17: unconnected-(U5-I14-Pad17) -> F_KEYS_3_14
- U7 pad 16: unconnected-(U7-I15-Pad16) -> F_KEYS_4_15
