File: keys.kicad_sch (KiCad schematic)
At the start: 168 parts, among them SW1 RotaryEncoder_Switch, U11 SLSS49E-3, U12 SLSS49E-3, U13 SLSS49E-3, U14 SLSS49E-3, U15 SLSS49E-3, U16 SLSS49E-3, U17 SLSS49E-3, U18 SLSS49E-3, U19 SLSS49E-3, U2 SLSS49E-3, U20 SLSS49E-3, U21 SLSS49E-3, U22 SLSS49E-3, U23 SLSS49E-3, U24 SLSS49E-3, U25 SLSS49E-3, U26 SLSS49E-3, U27 SLSS49E-3, U28 SLSS49E-3, U29 SLSS49E-3, U30 SLSS49E-3, U31 SLSS49E-3, U32 SLSS49E-3, U33 SLSS49E-3, U34 SLSS49E-3, U35 SLSS49E-3, U36 SLSS49E-3, U37 SLSS49E-3, U38 SLSS49E-3, U39 SLSS49E-3, U4 SLSS49E-3, U40 SLSS49E-3, U41 SLSS49E-3, U42 SLSS49E-3, U43 SLSS49E-3, U44 SLSS49E-3, U45 SLSS49E-3, U46 SLSS49E-3, U47 SLSS49E-3, U48 SLSS49E-3, U49 SLSS49E-3, U50 SLSS49E-3, U51 SLSS49E-3, U52 SLSS49E-3, U53 SLSS49E-3, U54 SLSS49E-3, U55 SLSS49E-3, U56 SLSS49E-3, U57 SLSS49E-3, U58 SLSS49E-3, U59 SLSS49E-3, U60 SLSS49E-3, U61 SLSS49E-3, U62 SLSS49E-3, U63 SLSS49E-3, U64 SLSS49E-3, U65 SLSS49E-3, U66 SLSS49E-3, U67 SLSS49E-3, U68 SLSS49E-3, U69 SLSS49E-3, U70 SLSS49E-3, U71 SLSS49E-3, U72 SLSS49E-3, U73 SLSS49E-3, U74 SLSS49E-3, U75 SLSS49E-3, U76 SLSS49E-3, U77 SLSS49E-3, U78 SLSS49E-3, U79 SLSS49E-3, U80 SLSS49E-3, U81 SLSS49E-3, U82 SLSS49E-3, U83 SLSS49E-3, U84 SLSS49E-3, U85 SLSS49E-3, U86 SLSS49E-3, U87 SLSS49E-3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

Commit message: second commit
Parts:
- removed S1, S2, S4: choc_stab, PCM_marbastlib-xp-choc:STAB_choc_2u, symbol PCM_marbastlib-choc:choc_stab
- added S1, S2, S3: MX_stab, PCM_marbastlib-mx:STAB_MX_ISO, symbol PCM_marbastlib-mx:MX_stab
- OLED: footprint (none) -> Connector_PinHeader_2.54mm:PinHeader_1x04_P2.54mm_Vertical
Connections:
- net +3V3: now also SW1.S1
- net GND: now also OLED.4 (Pin_4), SW1.C
- net ENCODER_A: now reaches SW1.A
- net ENCODER_B: now reaches SW1.B
- net ENCODER_SWITCH: now reaches SW1.S2
- net I2C1_SDA: now reaches OLED.1 (Pin_1)
- net I2C1_SCL: now reaches OLED.2 (Pin_2)
- net +5V: now reaches OLED.3 (Pin_3)

Commit message: bus
Parts:
- S2: renamed from S1; value MX_stab -> STAB_MX_ISO
- renumbered S2 to S1
Connections:
- net # renamed KEYS_3_12
- net ' renamed KEYS_3_11
- net , renamed KEYS_4_9
- net - renamed KEYS_1_11
- net . renamed KEYS_4_10
- net 0 renamed KEYS_1_10
- net 1 renamed KEYS_1_1
- net 2 renamed KEYS_1_2
- net 3 renamed KEYS_1_3
- net 4 renamed KEYS_1_4
- net 5 renamed KEYS_1_5
- net 6 renamed KEYS_1_6
- net 7 renamed KEYS_1_7
- net 8 renamed KEYS_1_8
- net 9 renamed KEYS_1_9
- net ; renamed KEYS_3_10
- net = renamed KEYS_1_12
- net A renamed KEYS_3_1
- net B renamed KEYS_4_6
- net BACKSPACE renamed KEYS_1_13
- net C renamed KEYS_4_4
- net CAPSLOCK renamed KEYS_3_0
- net D renamed KEYS_3_3
- net DELETE renamed KEYS_2_14
- net DOWN renamed KEYS_5_8
- net E renamed KEYS_2_3
- net ENCODER_SWITCH renamed KEYS_1_14
- net ENTER renamed KEYS_2_13
- net ESC renamed KEYS_0_0
- net F renamed KEYS_3_4
- net F1 renamed KEYS_0_1
- net F10 renamed KEYS_0_10
- net F11 renamed KEYS_0_11
- net F12 renamed KEYS_0_12
- net F2 renamed KEYS_0_2
- net F3 renamed KEYS_0_3
- net F4 renamed KEYS_0_4
- net F5 renamed KEYS_0_5
- net F6 renamed KEYS_0_6
- net F7 renamed KEYS_0_7
- net F8 renamed KEYS_0_8
- net F9 renamed KEYS_0_9
- net FN renamed KEYS_5_5
- net G renamed KEYS_3_5
- net H renamed KEYS_3_6
- net I renamed KEYS_2_8
- net J renamed KEYS_3_7
- net K renamed KEYS_3_8
- net L renamed KEYS_3_9
- net LALT renamed KEYS_5_2
- net LCTRL renamed KEYS_5_0
- net LEFT renamed KEYS_5_7
- net LSHIFT renamed KEYS_4_0
- net LWIN renamed KEYS_5_1
- net M renamed KEYS_4_8
- net N renamed KEYS_4_7
- net O renamed KEYS_2_9
- net P renamed KEYS_2_10
- net PGDN renamed KEYS_4_14
- net PGUP renamed KEYS_3_13
- net Q renamed KEYS_2_1
- net R renamed KEYS_2_4
- net RALT renamed KEYS_5_4
- net RCTRL renamed KEYS_5_6
- net RIGHT renamed KEYS_5_9
- net RSHIFT renamed KEYS_4_12
- net S renamed KEYS_3_2
- net SPACE renamed KEYS_5_3
- net T renamed KEYS_2_5
- net TAB renamed KEYS_2_0
- net U renamed KEYS_2_7
- net UP renamed KEYS_4_13
- net V renamed KEYS_4_5
- net W renamed KEYS_2_2
- net X renamed KEYS_4_3
- net Y renamed KEYS_2_6
- net Z renamed KEYS_4_2
- net [ renamed KEYS_2_11
- net \ renamed KEYS_4_1
- net ] renamed KEYS_2_12
- net ` renamed KEYS_1_0
- net / renamed KEYS_4_11
Other:
- moved on the sheet: S2, S3, U48

Commit message: assign footprints
Parts:
- C10, C11, C12, C13, C14, C15, C16, C17, C18, C19, C2, C20, C21, C22, C23, C24, C25, C26, C27, C28, C29, C3, C30, C31, C32, C33, C34, C35, C36, C37, C38, C39, C4, C40, C41, C42, C43, C44, C45, C46, C47, C48, C49, C5, C50, C51, C52, C53, C54, C55, C56, C57, C58, C59, C6, C60, C61, C62, C63, C64, C65, C66, C67, C68, C69, C7, C70, C71, C72, C73, C74, C75, C76, C77, C78, C79, C8, C80, C81, C82, C9: footprint (none) -> Capacitor_SMD:C_0402_1005Metric
- SW1: footprint (none) -> Rotary_Encoder:RotaryEncoder_Alps_EC11E-Switch_Vertical_H20mm
- U11, U12, U13, U14, U15, U16, U17, U18, U19, U2, U20, U21, U22, U23, U24, U25, U26, U27, U28, U29, U30, U31, U32, U33, U34, U35, U36, U37, U38, U39, U4, U40, U41, U42, U43, U44, U45, U46, U47, U48, U49, U50, U51, U52, U53, U54, U55, U56, U57, U58, U59, U60, U61, U62, U63, U64, U65, U66, U67, U68, U69, U70, U71, U72, U73, U74, U75, U76, U77, U78, U79, U80, U81, U82, U83, U84, U85, U86, U87, U88, U89: footprint Package_TO_SOT_SMD:SOT-23 -> MoonBoard:SLSS49E-3 with MX holes

Commit message: switch layout
Parts:
- removed S3: MX_stab, PCM_marbastlib-mx:STAB_MX_ISO, symbol PCM_marbastlib-mx:MX_stab
- added S83, S84: MX_stab, PCM_marbastlib-mx:STAB_MX_2.25u, symbol PCM_marbastlib-mx:MX_stab
- added U63 (x2): SLSS49E-3, MoonBoard:SLSS49E-3 with 2.25 MX holes, symbol MoonBoard:SLSS49E-3_with_switch
- added U63: SLSS49E-3, MoonBoard:SLSS49E-3 with 1.5u MX holes, symbol MoonBoard:SLSS49E-3_with_switch
- S27: renamed from S1; value MX_stab -> STAB_MX_2u; footprint PCM_marbastlib-mx:STAB_MX_ISO -> PCM_marbastlib-mx:STAB_MX_2u
- S3: value MX_stab -> STAB_MX_P_6.25U
- U11, U12, U13, U14, U15, U16, U17, U18, U19, U2, U20, U21, U22, U23, U24, U25, U26, U27, U28, U29, U30, U31, U32, U33, U34, U35, U36, U37, U38, U39, U4, U40, U41, U42, U43, U44, U45, U46, U47, U48, U50, U51, U52, U53, U54, U55, U56, U57, U58, U59, U60, U61, U63, U64, U65, U66, U67, U68, U69, U70, U71, U72, U73, U74, U77, U81, U82, U83, U84, U85, U86, U87, U88, U89: symbol Sensor_Magnetic:DRV5033AJxDBZ -> MoonBoard:SLSS49E-3_with_switch
- U49: footprint MoonBoard:SLSS49E-3 with MX holes -> MoonBoard:SLSS49E-3 with 1.5u MX holes; symbol Sensor_Magnetic:DRV5033AJxDBZ -> MoonBoard:SLSS49E-3_with_switch
- U62, U76: footprint MoonBoard:SLSS49E-3 with MX holes -> MoonBoard:SLSS49E-3 with 1.75u MX holes; symbol Sensor_Magnetic:DRV5033AJxDBZ -> MoonBoard:SLSS49E-3_with_switch
- U75, U78, U79, U80: footprint MoonBoard:SLSS49E-3 with MX holes -> MoonBoard:SLSS49E-3 with 1.25u MX holes; symbol Sensor_Magnetic:DRV5033AJxDBZ -> MoonBoard:SLSS49E-3_with_switch
- renumbered S2 to S41
Connections:
- net +3V3: now also U63.1 (VDD), U63.1 (VDD), U63.1 (VDD)
- net GND: now also U11.2 (GND), U12.2 (GND), U13.2 (GND), U14.2 (GND), U15.2 (GND), U16.2 (GND), U17.2 (GND), U18.2 (GND), U19.2 (GND), U2.2 (GND), U20.2 (GND), U21.2 (GND), U22.2 (GND), U23.2 (GND), U24.2 (GND), U25.2 (GND), U26.2 (GND), U27.2 (GND), U28.2 (GND), U29.2 (GND), U30.2 (GND), U31.2 (GND), U32.2 (GND), U33.2 (GND), U34.2 (GND), U35.2 (GND), U36.2 (GND), U37.2 (GND), U38.2 (GND), U39.2 (GND), U4.2 (GND), U40.2 (GND), U41.2 (GND), U42.2 (GND), U43.2 (GND), U44.2 (GND), U45.2 (GND), U46.2 (GND), U47.2 (GND), U48.2 (GND), U49.2 (GND), U50.2 (GND), U51.2 (GND), U52.2 (GND), U53.2 (GND), U54.2 (GND), U55.2 (GND), U56.2 (GND), U57.2 (GND), U58.2 (GND), U59.2 (GND), U60.2 (GND), U61.2 (GND), U62.2 (GND), U63.2 (GND), U64.2 (GND), U65.2 (GND), U66.2 (GND), U67.2 (GND), U68.2 (GND), U69.2 (GND), U70.2 (GND), U71.2 (GND), U72.2 (GND), U73.2 (GND), U74.2 (GND), U75.2 (GND), U76.2 (GND), U77.2 (GND), U78.2 (GND), U79.2 (GND), U80.2 (GND), U81.2 (GND), U82.2 (GND), U83.2 (GND), U84.2 (GND), U85.2 (GND), U86.2 (GND), U87.2 (GND), U88.2 (GND), U89.2 (GND), U63.2 (GND), U63.2 (GND), U63.2 (GND); no longer U11.3 (GND), U12.3 (GND), U13.3 (GND), U14.3 (GND), U15.3 (GND), U16.3 (GND), U17.3 (GND), U18.3 (GND), U19.3 (GND), U2.3 (GND), U20.3 (GND), U21.3 (GND), U22.3 (GND), U23.3 (GND), U24.3 (GND), U25.3 (GND), U26.3 (GND), U27.3 (GND), U28.3 (GND), U29.3 (GND), U30.3 (GND), U31.3 (GND), U32.3 (GND), U33.3 (GND), U34.3 (GND), U35.3 (GND), U36.3 (GND), U37.3 (GND), U38.3 (GND), U39.3 (GND), U4.3 (GND), U40.3 (GND), U41.3 (GND), U42.3 (GND), U43.3 (GND), U44.3 (GND), U45.3 (GND), U46.3 (GND), U47.3 (GND), U48.3 (GND), U49.3 (GND), U50.3 (GND), U51.3 (GND), U52.3 (GND), U53.3 (GND), U54.3 (GND), U55.3 (GND), U56.3 (GND), U57.3 (GND), U58.3 (GND), U59.3 (GND), U60.3 (GND), U61.3 (GND), U62.3 (GND), U63.3 (GND), U64.3 (GND), U65.3 (GND), U66.3 (GND), U67.3 (GND), U68.3 (GND), U69.3 (GND), U70.3 (GND), U71.3 (GND), U72.3 (GND), U73.3 (GND), U74.3 (GND), U75.3 (GND), U76.3 (GND), U77.3 (GND), U78.3 (GND), U79.3 (GND), U80.3 (GND), U81.3 (GND), U82.3 (GND), U83.3 (GND), U84.3 (GND), U85.3 (GND), U86.3 (GND), U87.3 (GND), U88.3 (GND), U89.3 (GND)
- net KEYS_0_0: now also U2.3 (VOUT); no longer U2.2 (OUT)
- net KEYS_0_1: now also U4.3 (VOUT); no longer U4.2 (OUT)
- net KEYS_0_10: now also U19.3 (VOUT); no longer U19.2 (OUT)
- net KEYS_0_11: now also U20.3 (VOUT); no longer U20.2 (OUT)
- net KEYS_0_12: now also U21.3 (VOUT); no longer U21.2 (OUT)
- net KEYS_0_2: now also U11.3 (VOUT); no longer U11.2 (OUT)
- net KEYS_0_3: now also U12.3 (VOUT); no longer U12.2 (OUT)
- net KEYS_0_4: now also U13.3 (VOUT); no longer U13.2 (OUT)
- net KEYS_0_5: now also U14.3 (VOUT); no longer U14.2 (OUT)
- net KEYS_0_6: now also U15.3 (VOUT); no longer U15.2 (OUT)
- net KEYS_0_7: now also U16.3 (VOUT); no longer U16.2 (OUT)
- net KEYS_0_8: now also U17.3 (VOUT); no longer U17.2 (OUT)
- net KEYS_0_9: now also U18.3 (VOUT); no longer U18.2 (OUT)
- net KEYS_1_0: now also U22.3 (VOUT); no longer U22.2 (OUT)
- net KEYS_1_1: now also U23.3 (VOUT); no longer U23.2 (OUT)
- net KEYS_1_10: now also U32.3 (VOUT); no longer U32.2 (OUT)
- net KEYS_1_11: now also U33.3 (VOUT); no longer U33.2 (OUT)
- net KEYS_1_12: now also U34.3 (VOUT); no longer U34.2 (OUT)
- net KEYS_1_13: now also U35.3 (VOUT); no longer U35.2 (OUT)
- net KEYS_1_2: now also U24.3 (VOUT); no longer U24.2 (OUT)
- net KEYS_1_3: now also U25.3 (VOUT); no longer U25.2 (OUT)
- net KEYS_1_4: now also U26.3 (VOUT); no longer U26.2 (OUT)
- net KEYS_1_5: now also U27.3 (VOUT); no longer U27.2 (OUT)
- net KEYS_1_6: now also U28.3 (VOUT); no longer U28.2 (OUT)
- net KEYS_1_7: now also U29.3 (VOUT); no longer U29.2 (OUT)
- net KEYS_1_8: now also U30.3 (VOUT); no longer U30.2 (OUT)
- net KEYS_1_9: now also U31.3 (VOUT); no longer U31.2 (OUT)
- net KEYS_2_0: now also U49.3 (VOUT); no longer U49.2 (OUT)
- net KEYS_2_1: now also U36.3 (VOUT); no longer U36.2 (OUT)
- net KEYS_2_10: now also U45.3 (VOUT); no longer U45.2 (OUT)
- net KEYS_2_11: now also U46.3 (VOUT); no longer U46.2 (OUT)
- net KEYS_2_12: now also U47.3 (VOUT); no longer U47.2 (OUT)
- net KEYS_2_13: now also U48.3 (VOUT); no longer U48.2 (OUT)
- net KEYS_2_14: now also U63.3 (VOUT); no longer U63.2 (OUT)
- net KEYS_2_2: now also U37.3 (VOUT); no longer U37.2 (OUT)
- net KEYS_2_3: now also U38.3 (VOUT); no longer U38.2 (OUT)
- net KEYS_2_4: now also U39.3 (VOUT); no longer U39.2 (OUT)
- net KEYS_2_5: now also U40.3 (VOUT); no longer U40.2 (OUT)
- net KEYS_2_6: now also U41.3 (VOUT); no longer U41.2 (OUT)
- net KEYS_2_7: now also U42.3 (VOUT); no longer U42.2 (OUT)
- net KEYS_2_8: now also U43.3 (VOUT); no longer U43.2 (OUT)
- net KEYS_2_9: now also U44.3 (VOUT); no longer U44.2 (OUT)
- net KEYS_3_0: now also U62.3 (VOUT); no longer U62.2 (OUT)
- net KEYS_3_1: now also U50.3 (VOUT); no longer U50.2 (OUT)
- net KEYS_3_10: now also U59.3 (VOUT); no longer U59.2 (OUT)
- net KEYS_3_11: now also U60.3 (VOUT); no longer U60.2 (OUT)
- net KEYS_3_12: now also U61.3 (VOUT); no longer U61.2 (OUT)
- net KEYS_3_13: now also U64.3 (VOUT); no longer U64.2 (OUT)
- net KEYS_3_2: now also U51.3 (VOUT); no longer U51.2 (OUT)
- net KEYS_3_3: now also U52.3 (VOUT); no longer U52.2 (OUT)
- net KEYS_3_4: now also U53.3 (VOUT); no longer U53.2 (OUT)
- net KEYS_3_5: now also U54.3 (VOUT); no longer U54.2 (OUT)
- net KEYS_3_6: now also U55.3 (VOUT); no longer U55.2 (OUT)
- net KEYS_3_7: now also U56.3 (VOUT); no longer U56.2 (OUT)
- net KEYS_3_8: now also U57.3 (VOUT); no longer U57.2 (OUT)
- net KEYS_3_9: now also U58.3 (VOUT); no longer U58.2 (OUT)
- net KEYS_4_0: now also U75.3 (VOUT); no longer U75.2 (OUT)
- net KEYS_4_1: now also U77.3 (VOUT); no longer U77.2 (OUT)
- net KEYS_4_10: now also U73.3 (VOUT); no longer U73.2 (OUT)
- net KEYS_4_11: now also U74.3 (VOUT); no longer U74.2 (OUT)
- net KEYS_4_12: now also U76.3 (VOUT); no longer U76.2 (OUT)
- net KEYS_4_13: now also U87.3 (VOUT); no longer U87.2 (OUT)
- net KEYS_4_14: now also U88.3 (VOUT); no longer U88.2 (OUT)
- net KEYS_4_2: now also U65.3 (VOUT); no longer U65.2 (OUT)
- net KEYS_4_3: now also U66.3 (VOUT); no longer U66.2 (OUT)
- net KEYS_4_4: now also U67.3 (VOUT); no longer U67.2 (OUT)
- net KEYS_4_5: now also U68.3 (VOUT); no longer U68.2 (OUT)
- net KEYS_4_6: now also U69.3 (VOUT); no longer U69.2 (OUT)
- net KEYS_4_7: now also U70.3 (VOUT); no longer U70.2 (OUT)
- net KEYS_4_8: now also U71.3 (VOUT); no longer U71.2 (OUT)
- net KEYS_4_9: now also U72.3 (VOUT); no longer U72.2 (OUT)
- net KEYS_5_0: now also U78.3 (VOUT); no longer U78.2 (OUT)
- net KEYS_5_1: now also U79.3 (VOUT); no longer U79.2 (OUT)
- net KEYS_5_2: now also U80.3 (VOUT); no longer U80.2 (OUT)
- net KEYS_5_3: now also U89.3 (VOUT); no longer U89.2 (OUT)
- net KEYS_5_4: now also U81.3 (VOUT); no longer U81.2 (OUT)
- net KEYS_5_5: now also U82.3 (VOUT); no longer U82.2 (OUT)
- net KEYS_5_6: now also U83.3 (VOUT); no longer U83.2 (OUT)
- net KEYS_5_7: now also U84.3 (VOUT); no longer U84.2 (OUT)
- net KEYS_5_8: now also U85.3 (VOUT); no longer U85.2 (OUT)
- net KEYS_5_9: now also U86.3 (VOUT); no longer U86.2 (OUT)
- new net KEYS_2_15: U63.3 (VOUT)
- new net KEYS_3_14: U63.3 (VOUT)
- new net KEYS_4_15: U63.3 (VOUT)
Other:
- note added: "ANSI ENTER"
- note added: "ANSI RSHIFT"
- note added: "ANSI \|"
- moved on the sheet: S3

Commit message: final key layout
Parts:
- S27: footprint PCM_marbastlib-mx:STAB_MX_2u -> PCM_marbastlib-mx:STAB_MX_P_2u
- S42: renamed from S41; footprint PCM_marbastlib-mx:STAB_MX_ISO -> PCM_marbastlib-mx:STAB_MX_P_ISO
- S57: renamed from S83; footprint PCM_marbastlib-mx:STAB_MX_2.25u -> PCM_marbastlib-mx:STAB_MX_P_2.25u
- S60: renamed from S84; footprint PCM_marbastlib-mx:STAB_MX_2.25u -> PCM_marbastlib-mx:STAB_MX_P_2.25u
- U48: footprint MoonBoard:SLSS49E-3 with MX holes -> MoonBoard:SLSS49E-3 with 1.5u MX holes
- U63: footprint MoonBoard:SLSS49E-3 with 2.25 MX holes -> MoonBoard:SLSS49E-3 with MX holes
- U63: footprint MoonBoard:SLSS49E-3 with 1.5u MX holes -> MoonBoard:SLSS49E-3 with MX holes
- U63: footprint MoonBoard:SLSS49E-3 with 2.25 MX holes -> MoonBoard:SLSS49E-3 with 1.25u MX holes
- U75: footprint MoonBoard:SLSS49E-3 with 1.25u MX holes -> MoonBoard:SLSS49E-3 with MX holes
Connections:
- net +5V: now also OLED.2 (Pin_2); no longer OLED.3 (Pin_3)
- net GND: now also OLED.1 (Pin_1); no longer OLED.4 (Pin_4)
- net I2C1_SCL: now also OLED.3 (Pin_3); no longer OLED.2 (Pin_2)
- net I2C1_SDA: now also OLED.4 (Pin_4); no longer OLED.1 (Pin_1)
Other:
- moved on the sheet: OLED, S42, S57, S60

Commit message: key filter
Parts:
- removed S57, S60: MX_stab, PCM_marbastlib-mx:STAB_MX_P_2.25u, symbol PCM_marbastlib-mx:MX_stab
- removed U63 (x2): SLSS49E-3, MoonBoard:SLSS49E-3 with MX holes, symbol MoonBoard:SLSS49E-3_with_switch
- removed U63: SLSS49E-3, MoonBoard:SLSS49E-3 with 1.25u MX holes, symbol MoonBoard:SLSS49E-3_with_switch
- U48: footprint MoonBoard:SLSS49E-3 with 1.5u MX holes -> MoonBoard:SLSS49E-3 with MX holes
- U75: footprint MoonBoard:SLSS49E-3 with MX holes -> MoonBoard:SLSS49E-3 with 1.25u MX holes
- renumbered S42 to S41
Other:
- note removed: "ANSI ENTER"
- note removed: "ANSI RSHIFT"
- note removed: "ANSI \|"

Commit message: rearrange LEDs
Parts:
- OLED: footprint Connector_PinHeader_2.54mm:PinHeader_1x04_P2.54mm_Vertical -> MoonBoard:OLED Module

Commit message: redo edge cuts
Parts:
- SW1: footprint Rotary_Encoder:RotaryEncoder_Alps_EC11E-Switch_Vertical_H20mm -> PCM_marbastlib-various:ROT_Alps_EC11E-Switch
Changed lines of the file:
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@@
       (effects (font (size 1.27 1.27)))
     )
-    (property "Footprint" "Rotary_Encoder:RotaryEncoder_Alps_EC11E-Switch_Vertical_H20mm" (at 365.76 59.436 0)
+    (property "Footprint" "PCM_marbastlib-various:ROT_Alps_EC11E-Switch" (at 365.76 59.436 0)
       (effects (font (size 1.27 1.27)) hide)
     )
