File: usb.kicad_sch (KiCad schematic)
At the start: 32 parts, among them J1 USB_A, J2 USB_A, J3 USB_C_Receptacle_USB2.0, U12 CH334U, U12 SRV05-4, U9 SRV05-4, Y3 12MHz

Commit message: add level shifter for rgb data line
Parts:
- removed C265, C268: 1u, Capacitor_SMD:C_0402_1005Metric, symbol Device:C_Small
- removed C266: 100n, Capacitor_SMD:C_0402_1005Metric, symbol Device:C_Small
- removed C267: 10u, Capacitor_SMD:C_0402_1005Metric, symbol Device:C_Small
- removed D2: SMF6.0CA, MoonBoard:SOD-123FL_L2.8-W1.8-LS3.7-BI, symbol Device:D_TVS
- removed F1, F2 (x2), F3: Polyfuse, Fuse:Fuse_1206_3216Metric, symbol Device:Polyfuse
- removed FB1 (x2), FB2 (x2): 100R@100MHz, Inductor_SMD:L_0805_2012Metric, symbol Device:FerriteBead_Small
- removed H1, H2, H3, H4: MountingHole_Pad, symbol Mechanical:MountingHole_Pad
- removed J1, J2: USB_A, MoonBoard:USB-A-SMD_AF-APPLE-10.6, symbol Connector:USB_A
- removed J3 (x2): USB_C_Receptacle_USB2.0, MoonBoard:HRO-TYPE-C-31-M-12-Assembly, symbol Connector:USB_C_Receptacle_USB2.0
- removed R92, R93: 56k, Resistor_SMD:R_0402_1005Metric, symbol Device:R_Small
- removed R94, R95: 5k1, Resistor_SMD:R_0402_1005Metric, symbol Device:R_Small
- removed U12, U9: SRV05-4, PCM_marbastlib-various:SOT-23-6-routable, symbol PCM_marbastlib-various:SRV05-4
- removed U12: CH334U, Package_SO:SSOP-28_3.9x9.9mm_P0.635mm, symbol MoonBoard:CH334U
- removed USB1 (x3): X1224WRS-04-LPV01, Connector_Molex:Molex_Pico-EZmate_78171-0004_1x04-1MP_P1.20mm_Vertical, symbol Connector:Conn_01x04_Socket
- removed Y3: 12MHz, Crystal:Crystal_SMD_3225-4Pin_3.2x2.5mm, symbol Device:Crystal_GND24
Connections:
- no-connect marks 8 -> 0
