File: MoonBoard.kicad_sch (KiCad schematic)
At the start: 46 parts, among them SW1 SW_SPST, U1 AMS1117-3.3, U2 STM32F446RETx, U3 H5VU25U, U9 SN74LV1T34DBV, Y1 25MHz

Commit message: f303
Parts:
- removed C10: 2u2, Capacitor_SMD:C_0603_1608Metric, symbol Device:C_Small
- removed U2: STM32F446RETx, Package_QFP:LQFP-64_10x10mm_P0.5mm, symbol MCU_ST_STM32F4:STM32F446RETx
- removed U3 (x2): H5VU25U, MoonBoard:DFN2510, symbol Unified-Daughterboard-rescue:TPD4E05U06DQAR-acheronSymbols
- removed Y1: 25MHz, Crystal:Crystal_SMD_3225-4Pin_3.2x2.5mm, symbol Device:Crystal_GND24
- added C19, C265: 2u2, symbol Device:C_Small
- added FB1, FB2: 120R @ 100MHz, symbol Device:FerriteBead_Small
- added U2: STM32F303CBTx, Package_QFP:LQFP-48_7x7mm_P0.5mm, symbol MCU_ST_STM32F3:STM32F303CBTx
- added X1: 8MHz, Crystal:Crystal_SMD_HC49-SD, symbol Device:Crystal
- added X2: 32.768kHz, symbol Device:Crystal
- C3, C4: value 14p -> C_Small; footprint Capacitor_SMD:C_0402_1005Metric -> (none)
- C9: value 100n -> 1u
Connections:
- net +3V3: now also FB1.1, U2.1 (VBAT), U2.24 (VDD), U2.36 (VDD), U2.48 (VDD); no longer C11.1, C12.1
- net +5V: now also C265.2, FB2.1; no longer USB1.1 (Pin_1)
- net BOOT0: now also U2.44 (BOOT0)
- net GND: now also C3.1, C4.1, C19.1, C265.1, U2.23 (VSS), U2.35 (VSS), U2.47 (VSS), U2.8 (VSSA); no longer C3.2, C4.2
- net I2C1_SCL: now also U2.42 (PB6), U2.45 (PB8)
- net I2C1_SDA: now also U2.43 (PB7), U2.46 (PB9)
- net OSC_IN: now also C3.2, U2.5 (PF0), X1.2; no longer C3.1
- net OSC_OUT: now also C4.2, U2.6 (PF1), X1.1; no longer C4.1
- net SWCLK: now also U2.37 (PA14)
- net SWDIO: now also U2.34 (PA13)
- net SWO: now also U2.39 (PB3)
- net USB_D+: now also U2.33 (PA12)
- net USB_D-: now also U2.32 (PA11)
- net ~{RESET}: now also U2.7 (NRST)
- net BUZZ+ renamed DAC1_OUT1
- net DAC1_OUT1: now also U2.14 (PA4)
- net BUZZ- renamed DAC1_OUT2
- net DAC1_OUT2: now also U2.15 (PA5)
- new net: C19.2, FB2.2, USB1.1 (Pin_1)
- new net +3.3VADC: C11.1, C12.1, FB1.2, U2.9 (VDDA)
- new net ADC1_IN1: U2.10 (PA0)
- new net ADC1_IN2: U2.11 (PA1)
- new net ADC1_IN3: U2.12 (PA2)
- new net ADC1_IN4: U2.13 (PA3)
- new net ADC2_IN3: U2.16 (PA6)
- new net ADC2_IN4: U2.17 (PA7)
- new net ADC3_IN1: U2.19 (PB1)
- new net ADC3_IN3: U2.25 (PB12)
- new net ADC3_IN5: U2.26 (PB13)
- new net ADC4_IN4: U2.27 (PB14)
- new net ADC4_IN5: U2.28 (PB15)
- new net OSC32_IN: U2.3 (PC14)
- new net OSC32_OUT: U2.4 (PC15)
- no-connect marks 29 -> 0
Other:
- note removed: "MCU Decoupling"
- moved on the sheet: BZ1, C11, C12, C5, C6, C7, C8, R1, SW1, U9, USB1

Commit message: change HSE
Parts:
- removed D2: 1N4148WS, Diode_SMD:D_SOD-323, symbol Diode:1N4148WS
- removed X1: 8MHz, Crystal:Crystal_SMD_HC49-SD, symbol Device:Crystal
- added C10, C266: 15p, symbol Device:C_Small
- added R96: 0, symbol Device:R_Small
- added R97, R98: 1, Resistor_SMD:R_1206_3216Metric, symbol Device:R_Small
- added Y1: 16MHz, Crystal:Crystal_SMD_3225-4Pin_3.2x2.5mm, symbol Device:Crystal_GND24
- C2: footprint Capacitor_Tantalum_SMD:CP_EIA-3528-21_Kemet-B -> Capacitor_SMD:C_1206_3216Metric
- C3, C4: value C_Small -> 8p
- FB1, FB2: footprint (none) -> Inductor_SMD:L_0805_2012Metric
- Y2: renamed from X2; footprint (none) -> Crystal:Crystal_C38-LF_D3.0mm_L8.0mm_Horizontal
Connections:
- net GND: now also C10.1, C266.1, R97.2, R98.2, Y1.2, Y1.4; no longer C1.2, C2.2, H2.1, H3.1, H4.1, H5.1, H6.1, H7.1, H8.1
- net OSC32_IN: now also Y2.1, C10.2
- net OSC32_OUT: now also Y2.2, C266.2
- net OSC_IN: now also Y1.1
- net OSC_OUT: now also R96.1; no longer C4.2
- new net: C2.2, R98.1
- new net: C1.2, R97.1
- new net: C4.2, R96.2, Y1.3
- no-connect marks 0 -> 7
Other:
- note added: "9pF"
- note added: "~12.5pF"
- moved on the sheet: C1, C2, C3, C4, NT1, NT2, U1, Y2

Commit message: f303 routing
Parts:
- removed C10, C266: 15p, symbol Device:C_Small
- removed U9: SN74LV1T34DBV, Package_TO_SOT_SMD:SOT-23-5, symbol Logic_LevelTranslator:SN74LV1T34DBV
- removed Y2: 32.768kHz, Crystal:Crystal_C38-LF_D3.0mm_L8.0mm_Horizontal, symbol Device:Crystal
- added C12: 100n, Capacitor_SMD:C_0402_1005Metric, symbol Device:C_Small
- added J1: AudioJack4, Connector_Audio:Jack_3.5mm_PJ320E_Horizontal, symbol Connector_Audio:AudioJack4
- added U2: 74LS08, Package_SO:SOIC-14_3.9x8.7mm_P1.27mm, symbol 74xx:74LS08
- C1: renamed from C19; footprint (none) -> Capacitor_SMD:C_0805_2012Metric
- C13: renamed from C3; footprint (none) -> Capacitor_SMD:C_0402_1005Metric
- C14: renamed from C4; footprint (none) -> Capacitor_SMD:C_0402_1005Metric
- C2: renamed from C265; footprint (none) -> Capacitor_SMD:C_0805_2012Metric
- R1: renamed from R92; footprint Resistor_SMD:R_0402_1005Metric -> Resistor_SMD:R_0603_1608Metric
- R2: renamed from R93; footprint Resistor_SMD:R_0402_1005Metric -> Resistor_SMD:R_0603_1608Metric
- R3: renamed from R91; footprint Resistor_SMD:R_0402_1005Metric -> Resistor_SMD:R_0603_1608Metric
- R8: renamed from R96; footprint (none) -> Resistor_SMD:R_0603_1608Metric_Pad0.98x0.95mm_HandSolder
- renumbered C12 to C10, C9 to C11, C1 to C3, C2 to C4, C11 to C9, FB2 to FB1, FB1 to FB2, H5 to H2, H2 to H3, H6 to H4, H3 to H5, H7 to H6, H4 to H7, R97 to R4, R98 to R5, R94 to R6, R95 to R7, R1 to R9, U2 to U3
Connections:
- net ADC3_IN1 is gone; now on net S2: U3.19 (PB1)
- net +3V3: now also SWD1.5 (Pin_5); no longer SWD1.3 (Pin_3)
- net +5V: now also C12.1, J1.T, U2.14 (VCC)
- net GND: now also H5.1, SWD1.3 (Pin_3), C12.2, J1.S, U2.7 (GND); no longer H1.1, SWD1.4 (Pin_4)
- net I2C1_SCL: no longer U3.45 (PB8)
- net I2C1_SDA: no longer U3.46 (PB9)
- net S0: now also U3.22 (PB11)
- net S1: now also U3.21 (PB10)
- net S3: now also U3.20 (PB2)
- net SWCLK: now also R2.1; no longer R1.2
- net SWO: now also R1.2; no longer R2.1
- net VBUS: now reaches C1.2, FB1.2, USB1.1 (Pin_1)
- net at R2.2: now also SWD1.4 (Pin_4); no longer SWD1.5 (Pin_5)
- net at R9.1: now also U2.11
- net out_esr: now reaches C4.2, R5.1
- net in_esr: now reaches C3.2, R4.1
- net USART1_CK: now reaches U3.29 (PA8)
- net USART1_TX: now reaches U3.30 (PA9)
- net USART1_TX: now also J1.R1
- net USART1_RX: now reaches U3.31 (PA10)
- net USART1_RX: now also J1.R2
- net TIM8_CH1: now reaches U3.38 (PA15)
- net TIM8_CH1: now also U2.12, U2.13
- net ADC1_IN1: no longer names the net of U3.10 (PA0)
- net ADC1_IN2: no longer names the net of U3.11 (PA1)
- net ADC3_IN3 renamed ADC4_IN3
- net ADC3_IN5: no longer names the net of U3.26 (PB13)
- net ADC4_IN5: no longer names the net of U3.28 (PB15)
- net OSC32_IN: no longer names the net of U3.3 (PC14)
- net OSC32_OUT: no longer names the net of U3.4 (PC15)
- no-connect marks 7 -> 16
Other:
- note added: ""Level Shifter""
- note removed: "Level Shifter"
- note removed: "~12.5pF"
- moved on the sheet: BZ1, C10, C11, C13, C14, C3, C5, C6, C7, C8, C9, FB2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

Commit message: dip switch
Parts:
- added SW2: SW_DIP_x04, Button_Switch_THT:SW_DIP_SPSTx04_Slide_6.7x11.72mm_W7.62mm_P2.54mm_LowProfile, symbol Switch:SW_DIP_x04
- BZ1: value Buzzer -> AST1109MLTRQ
- H1, H2, H3, H4, H5, H6, H7, H8, TH1, TH2, TH3: now left out of the parts list
- J1: value AudioJack4 -> TRRS
- R6, R7: footprint Resistor_SMD:R_0402_1005Metric -> Resistor_SMD:R_0603_1608Metric
Connections:
- net ENCODER_A: now also U3.2 (PC13)
- net ENCODER_B: now also U3.3 (PC14)
- net ENCODER_SW: now also ENCODER1.S1, U3.18 (PB0); no longer ENCODER1.S2
- net GND: now also ENCODER1.S2, SW2.1, SW2.2, SW2.3, SW2.4; no longer ENCODER1.S1
- net SW_DIP_0: now reaches U3.10 (PA0)
- net SW_DIP_0: now also SW2.8
- net SW_DIP_3: now reaches U3.11 (PA1)
- net SW_DIP_3: now also SW2.5
- net SW_DIP_2: now reaches U3.26 (PB13)
- net SW_DIP_2: now also SW2.6
- net SW_DIP_1: now reaches U3.28 (PB15)
- net SW_DIP_1: now also SW2.7
Other:
- note added: "DIP Selector Switch"
- note added: "JLCPCB Tooling"
- note added: "Serial USART TRRS"
- note added: "Unused AND Gates"
- note removed: "Crystal"
- moved on the sheet: BZ1, C1, C10, C11, C12, C13, C14, C2, C5, C6, C7, C8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
